File: USB-PD-Power-Supply.kicad_sch (KiCad schematic)
At the start: 40 parts, among them IC1 MC14051BDR2G, J1 Screw_Terminal_01x02, J2 USB_C_Receptacle_USB2.0_16P, J3 Conn_01x03_Pin, Q1 2N7002, U1 SW-SMD_DSHP03TS-S, U2 CH224A, U3 TPS70933DBVR

Commit message: Completed Routing, Adjusted Silkscreen, and Images
Connections:
- net CFB1: now also IC1.9 (C); no longer IC1.11 (A)
- net CFB3_SDA: now also IC1.11 (A); no longer IC1.9 (C)
- net GND: now also J1.1 (Pin_1); no longer J1.2 (Pin_2)
- net USB_N: now also D2.1, J2.A7 (D-), J2.B7 (D-), U2.5 (DM); no longer D3.1, J2.A6 (D+), J2.B6 (D+), U2.4 (DP)
- net USB_P: now also D3.1, J2.A6 (D+), J2.B6 (D+), U2.4 (DP); no longer D2.1, J2.A7 (D-), J2.B7 (D-), U2.5 (DM)
- net V_USB: now also J1.2 (Pin_2); no longer J1.1 (Pin_1)
Changed lines of the file:
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@@
 	)
 	(label "CFB1"
-		(at 336.55 157.48 0)
+		(at 336.55 162.56 0)
 		(effects
 			(font
@@
 	)
 	(label "CFB3_SDA"
-		(at 336.55 162.56 0)
+		(at 336.55 157.48 0)
 		(effects
 			(font
@@
 		)
 	)
-	(label "USB_N"
+	(label "USB_P"
 		(at 161.29 88.9 0)
 		(effects
@@
 		)
 	)
-	(label "USB_P"
+	(label "USB_N"
 		(at 161.29 86.36 0)
 		(effects
@@
 	(symbol
 		(lib_id "Connector:Screw_Terminal_01x02")
-		(at 358.14 78.74 0)
+		(at 358.14 81.28 0)
+		(mirror x)
 		(unit 1)
 		(body_style 1)
@@
 		(in_pos_files yes)
 		(dnp no)
-		(fields_autoplaced yes)
 		(property "Reference" "J1"
-			(at 360.68 78.7399 0)
+			(at 360.68 81.2801 0)
 			(show_name no)
 			(do_not_autoplace no)
@@
 		)
 		(property "Value" "Screw_Terminal_01x02"
-			(at 360.68 81.2799 0)
+			(at 360.68 78.7401 0)
 			(show_name no)
 			(do_not_autoplace no)
@@
 		)
 		(property "Footprint" "TerminalBlock_Phoenix:TerminalBlock_Phoenix_MKDS-1,5-2-5.08_1x02_P5.08mm_Horizontal"
-			(at 358.14 78.74 0)
+			(at 358.14 81.28 0)
 			(hide yes)
 			(show_name no)
@@
 		)
 		(property "Datasheet" ""
-			(at 358.14 78.74 0)
+			(at 358.14 81.28 0)
 			(hide yes)
 			(show_name no)
@@
 		)
 		(property "Description" "Generic screw terminal, single row, 01x02, script generated (kicad-library-utils/schlib/autogen/connector/)"
-			(at 358.14 78.74 0)
+			(at 358.14 81.28 0)
 			(hide yes)
 			(show_name no)
